Commit message: fix: hand offset

File: assets/unitree_hand/unitree_dex3_left.urdf (robot description, URDF)
Before this commit: robot dex3_left, 15 links, 14 joints
Joints:
- joint left_hand_thumb_0_joint: limit lower=-1.04719755 upper=1.04719755 effort=2.45 velocity=6.857 -> lower=-2.443461 upper=0.174533 effort=2.45 velocity=6.857

File: assets/unitree_hand/unitree_dex3_right.urdf (robot description, URDF)
Before this commit: robot dex3_right, 15 links, 14 joints
Joints:
- joint right_hand_thumb_0_joint: limit lower=-1.04719755 upper=1.04719755 effort=2.45 velocity=6.857 -> lower=-2.443461 upper=0.174533 effort=2.45 velocity=6.857
